File: AudioDSP/VirtualSense_ADSP.sch (KiCad schematic (older format))
At the start: 50 parts, among them M1 MIC, P2 CONN_1, P3 CONN_1, P5 CONN_1, P6 CONN_1, P7 DSP, P8 uC, U2 TLV320AIC3204, U4 DSX321G_12MHZ

Commit message: create schematics, components footprints, board layout.
Parts:
- removed BT1: WAKEUP, symbol SW_PUSH
- removed C1: 1u, symbol CP1SMALL
- removed C? (x2): 47pF, symbol CSMALL
- removed CONN2, CONN4: CONN_14, symbol CONN_14
- removed CONN2: 4V5, symbol CONN_2
- removed JP1: USB-3V3, symbol BREAKER
- removed M1: MIC, symbol SPEAKER
- removed P7: DSP, symbol CONN_1
- removed R? (x2): 33, symbol RSML
- removed USB1: USB-PLUG, symbol CONN_4
- added BT2: 18650, symbol BH2466
- added BTB1: 1V3, symbol BATTERY
- added BTB1-2: BH411-1P, symbol BH2466
- added C1, C2, C3: 470n, symbol CSMALL
- added C10, C12, C13, C14, C16: NO, symbol CSMALL
- added C17: 10u, symbol CP1SMALL
- added C20: 100n, symbol CSMALL
- added D5: ZMM5234B-7-F, symbol ZENERSMALL
- added JP1: 3V3-USB, symbol JUMPER
- added P10, P11: DSP-SDA, symbol CONN_1
- added P12, P20, P9: CONN_1, symbol CONN_1
- added P3: CH1, symbol CONN_2
- added P4: CH2, symbol CONN_2
- added P5: CH3, symbol CONN_2
- added PBT1: WAKEUP, symbol PUSH-BT_4
- added R10, R9: 0, symbol RSML
- added R11: 300, symbol RSML
- added R23: 100K, symbol RSML
- added R4, R5, R6, R8: 1K, symbol RSML
- added USB1: MICRO-USB, symbol USB-REC
- BT1: value BH2466 -> 18650
- C6: value NO -> 470n
- P2: renamed from P8; value uC -> DSP
- R1: value 2K2 -> 1K
- gave numbers to parts that had none: 4
- renumbered CONN1 to P1, P2 to P13, P3 to P14, P5 to P7, P6 to P8
Connections:
- net labels added: 1V3, 3V6_BAT, CH1_N, CH1_P, CH2_N, CH2_P, CH3_N, CH3_P, MICBIAS, USB_CLK_12MHZ
- net labels removed: 3V3L, 4V5, ADC0/P6.0, ADC1/P6.1, ADC2/P6.2, ADC3/P6.3, ADC4/P6.4, ADC5/P6.5, ADC6/P6.6, CLKOUT, DIO2/P8.5, DIO3/P8.6, GND, INT0/P2.0, INT1/P2.3, INT2/P2.5, INT3/P2.6, INT4/P2.7, LED0/P8.0, LED1/P8.1, LED2/P8.2, MICN, MICP, RXD2/MISO3/P5.7, SCL/P3.2, SDA/P3.1, SN0_EN/P8.3, SN1_EN/P8.4, TARGET_PWR_GOOD, TXD2/MOSI3/P5.6, VREF+/P5.0, VREF-/P5.1
- wire segments 166 -> 171
- no-connect marks 19 -> 20
Other:
- note added: "1DAY BATTERY-PACK"
- note added: "BIOS BATTERY(RTC)"
- note added: "INPUT CHANNELS"
- note added: "Idrophone PCB Layout"
- moved on the sheet: C11, C18, C21, C29, C7, DJ2235, P13, P14, P2, P7, P8, R12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

Commit message: add too many libraries on schematics, board disposal almolst complete, hope that will be routed
Parts:
- removed C29: 1u, symbol CP1SMALL
- removed DJ2235: SW1, symbol SWITCH_DJ2235
- added C39, C51: 10u, symbol CP1SMALL
- added C48: 68n, symbol CSMALL
- added C49: 100n, symbol CSMALL
- added C50: 4u7, symbol CP1SMALL
- added C62: 1u, symbol CP1SMALL
- added D10, D11, D6, D7, D8, D9: LED, symbol LED
- added P22: SYS-LOAD, symbol CONN_1
- added P6: DC-IN, symbol CONN_2
- added R55, R62, R63, R64, R65, R66: 220, symbol RSML
- added R56, R57, R60, R67: 10K, symbol RSML
- added R58: 1K5, symbol RSML
- added R59: 3K, symbol RSML
- added R61: 100K, symbol RSML
- added SW1: SSSS224001, symbol SSSS224001
- added TH1: NTHS0603N01N1003JE, symbol THERMISTOR
- added U6: MAX8934, symbol MAX8934
Connections:
- net labels added: CHARGE_LDO, CHARGE_OUT
- wire segments 171 -> 244
- no-connect marks 20 -> 21
Other:
- note added: "BATTERY CHARGER"
- moved on the sheet: R10, R11, R14, U4

Commit message: Schematic and board complete (add tps60125 charge-pump, tps77533 LDO regolator, oled).
Parts:
- removed BT1, BT2: 18650, symbol BH2466
- removed BTB1: 1V3, symbol BATTERY
- removed BTB1-2: BH411-1P, symbol BH2466
- removed C11, C17, C21, C39, C51, C7: 10u, symbol CP1SMALL
- removed C13, C8: NO, symbol CSMALL
- removed C18, C62: 1u, symbol CP1SMALL
- removed C2: 470n, symbol CSMALL
- removed C23, C50: 4u7, symbol CP1SMALL
- removed C48: 68n, symbol CSMALL
- removed C49: 100n, symbol CSMALL
- removed D10, D11, D6, D7, D8, D9: LED, symbol LED
- removed P10, P11: DSP-SDA, symbol CONN_1
- removed P22: SYS-LOAD, symbol CONN_1
- removed P6: DC-IN, symbol CONN_2
- removed PBT1: WAKEUP, symbol PUSH-BT_4
- removed R1, R2: 1K, symbol RSML
- removed R12, R35: 0, symbol RSML
- removed R15: 2, symbol RSML
- removed R55, R62, R63, R64, R65, R66: 220, symbol RSML
- removed R56, R57, R60, R67: 10K, symbol RSML
- removed R58: 1K5, symbol RSML
- removed R59: 3K, symbol RSML
- removed R61: 100K, symbol RSML
- removed SW1: SSSS224001, symbol SSSS224001
- removed TH1: NTHS0603N01N1003JE, symbol THERMISTOR
- removed U6: MAX8934, symbol MAX8934
- added C11, C17, C2, C21, C7: 10u, symbol CBIG
- added C18: 4u7, symbol CBIG
- added C69: NO, symbol CP1
- added P1: 3V3, symbol CONN_2
- added SW1: JS202011SCQN, symbol JS202011SCQN
- added U7: TPS77533, symbol TPS77533
- C1: value 470n -> 100n
- P6: renamed from P1; value 3V3 -> 3V3-REG
- U4: value DSX321G_12MHZ -> ASDM1-12.000MHZ
Connections:
- net labels removed: 1V3, 3V6_BAT, CHARGE_LDO, CHARGE_OUT, DSP_WAKEUP
- wire segments 244 -> 158
- no-connect marks 21 -> 23
Other:
- note removed: "1DAY BATTERY-PACK"
- note removed: "BATTERY CHARGER"
- note removed: "BIOS BATTERY(RTC)"
- moved on the sheet: JP1, L1, L2, L3, P3, P5, P6, R10, R11, R14, U1, U4

Commit message: gerber and schematic modified, sendt to MCE
Parts:
- added P10: AIC-CLK, symbol CONN_1
- added P11, P22: CONN_1, symbol CONN_1
Connections:
- wire segments 158 -> 165
- no-connect marks 23 -> 21
Other:
- moved on the sheet: P12, P13, P14, P7, P8, P9, SW1
