File: AudioDSP/VirtualSense_ADSP_2.sch (KiCad schematic (older format))
At the start: 29 parts, among them P10 DSP-SDA, P11 DSP-SCL, U5 C5535, X1 32.768KHz

Commit message: create schematics, components footprints, board layout.
Parts:
- removed BT1: 1V3, symbol BATTERY
- removed D? (x3): LED, symbol LED
- removed P10: DSP-SDA, symbol CONN_1
- removed P11: DSP-SCL, symbol CONN_1
- removed R? (x3): 220, symbol RSML
- added C30: 10u, symbol CP1SMALL
- added C38: 100n, symbol CSMALL
- added C39: 1n, symbol CSMALL
- added D2, D3, D4: LED, symbol LED
- added JP2: LED-DEBUG, symbol JUMPER
- added L4: BLM18AG601SN1D, symbol FILTER
- added P15: GPIOS, symbol CONN_5
- added P16: SPI, symbol CONN_9
- added P17: UART, symbol CONN_4
- added P18: I2C, symbol CONN_4
- added P21: DSP-SDA, symbol CONN_1
- added PBT2: STATUS, symbol PUSH-BT_4
- added R25, R26, R48: 0, symbol RSML
- added R28, R32, R49: 220, symbol RSML
- D0: renamed from D1; value LED -> NO
- R16: value 220 -> NO
- gave numbers to parts that had none: 3
Connections:
- net labels added: 1V3, 3V3_USB, GPIO0, GPIO1, GPIO2, LED1, LED2, LED3, LED4, SD1_CLK, SD1_CMD, SD1_DATA0, SD1_DATA1, SD1_DATA2, SD1_DATA3, SD2_CLK, SD2_CMD, SD2_DATA0, SD2_DATA1, SD2_DATA2, SD2_DATA3, SPI_CLK, SPI_CS0, SPI_CS1, SPI_CS2, SPI_CS3, SPI_RX, SPI_TX, UART_RXD, UART_TXD, USB_CLK_12MHZ, USB_N, USB_P, VUSB
- net labels removed: DIO1/P7.5, RXD2/MISO3/P5.7, SD_CLK, SD_CMD, SD_DATA0, SD_DATA1, SD_DATA2, SD_DATA3, TARGET_PWR_GOOD, TXD2/MOSI3/P5.6
- wire segments 98 -> 159
- no-connect marks 35 -> 19
Other:
- moved on the sheet: D0, D1, R16, R17, R18, R19, R20, R21, R22, R24, R27, R33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

Commit message: add too many libraries on schematics, board disposal almolst complete, hope that will be routed
Parts:
- removed C39: 1n, symbol CSMALL
- added C29: 100n, symbol CSMALL
- added R54: 0, symbol RSML
- added U3: SI7020, symbol SI7020
Connections:
- wire segments 159 -> 167
- no-connect marks 19 -> 21
Other:
- moved on the sheet: R48
Changed lines of the file:
@@
 NoConn ~ 1900 1900
 $Comp
-L GNDPWR #PWR049
+L GNDPWR #PWR056
 U 1 1 521E22FA
 P 1400 2150
-F 0 "#PWR049" H 1400 2200 40  0001 C CNN
+F 0 "#PWR056" H 1400 2200 40  0001 C CNN
 F 1 "GNDPWR" H 1400 2070 40  0000 C CNN
 F 2 "" H 1400 2150 60  0001 C CNN
@@
 $EndComp
 $Comp
-L GNDPWR #PWR050
+L GNDPWR #PWR057
 U 1 1 521E27C4
 P 900 6650
-F 0 "#PWR050" H 900 6700 40  0001 C CNN
+F 0 "#PWR057" H 900 6700 40  0001 C CNN
 F 1 "GNDPWR" H 900 6570 40  0000 C CNN
 F 2 "" H 900 6650 60  0001 C CNN
@@
 $EndComp
 $Comp
-L 3V3 #PWR051
+L 3V3 #PWR058
 U 1 1 521E2923
 P 850 5750
-F 0 "#PWR051" H 850 5850 40  0001 C CNN
+F 0 "#PWR058" H 850 5850 40  0001 C CNN
 F 1 "3V3" H 850 5875 40  0000 C CNN
 F 2 "" H 850 5750 60  0001 C CNN
@@
 $EndComp
 $Comp
-L GNDPWR #PWR052
+L GNDPWR #PWR059
 U 1 1 521E2CF9
 P 1850 5950
-F 0 "#PWR052" H 1850 6000 40  0001 C CNN
+F 0 "#PWR059" H 1850 6000 40  0001 C CNN
 F 1 "GNDPWR" H 1850 5870 40  0000 C CNN
 F 2 "" H 1850 5950 60  0001 C CNN
@@
 $EndComp
 $Comp
-L GNDPWR #PWR053
+L GNDPWR #PWR060
 U 1 1 521E2F5E
 P 1100 5300
-F 0 "#PWR053" H 1100 5350 40  0001 C CNN
+F 0 "#PWR060" H 1100 5350 40  0001 C CNN
 F 1 "GNDPWR" H 1100 5220 40  0000 C CNN
 F 2 "" H 1100 5300 60  0001 C CNN
@@
 L CSMALL C24
 U 1 1 521E31D3
-P 1500 4950
-F 0 "C24" H 1525 5000 30  0000 L CNN
-F 1 "100n" H 1525 4900 30  0000 L CNN
-F 2 "" H 1500 4950 60  0000 C CNN
-F 3 "" H 1500 4950 60  0000 C CNN
-	1    1500 4950
-	1    0    0    -1
-$EndComp
-$Comp
-L 3V3 #PWR054
+P 1550 5000
+F 0 "C24" H 1575 5050 30  0000 L CNN
+F 1 "100n" H 1575 4950 30  0000 L CNN
+F 2 "" H 1550 5000 60  0000 C CNN
+F 3 "" H 1550 5000 60  0000 C CNN
+	1    1550 5000
+	1    0    0    -1
+$EndComp
+$Comp
+L 3V3 #PWR061
 U 1 1 521E31D9
-P 1500 4800
-F 0 "#PWR054" H 1500 4900 40  0001 C CNN
-F 1 "3V3" H 1500 4925 40  0000 C CNN
-F 2 "" H 1500 4800 60  0001 C CNN
-F 3 "" H 1500 4800 60  0001 C CNN
-	1    1500 4800
-	1    0    0    -1
-$EndComp
-$Comp
-L GNDPWR #PWR055
+P 1300 4700
+F 0 "#PWR061" H 1300 4800 40  0001 C CNN
+F 1 "3V3" H 1300 4825 40  0000 C CNN
+F 2 "" H 1300 4700 60  0001 C CNN
+F 3 "" H 1300 4700 60  0001 C CNN
+	1    1300 4700
+	1    0    0    -1
+$EndComp
+$Comp
+L GNDPWR #PWR062
 U 1 1 521E31DF
-P 1500 5100
-F 0 "#PWR055" H 1500 5150 40  0001 C CNN
-F 1 "GNDPWR" H 1500 5020 40  0000 C CNN
-F 2 "" H 1500 5100 60  0001 C CNN
-F 3 "" H 1500 5100 60  0001 C CNN
-	1    1500 5100
+P 1550 5150
+F 0 "#PWR062" H 1550 5200 40  0001 C CNN
+F 1 "GNDPWR" H 1550 5070 40  0000 C CNN
+F 2 "" H 1550 5150 60  0001 C CNN
+F 3 "" H 1550 5150 60  0001 C CNN
+	1    1550 5150
 	1    0    0    -1
 $EndComp
@@
 NoConn ~ 1900 4900
 $Comp
-L GNDPWR #PWR056
+L GNDPWR #PWR063
 U 1 1 521E336E
 P 1400 4350
-F 0 "#PWR056" H 1400 4400 40  0001 C CNN
+F 0 "#PWR063" H 1400 4400 40  0001 C CNN
 F 1 "GNDPWR" H 1400 4270 40  0000 C CNN
 F 2 "" H 1400 4350 60  0001 C CNN
@@
 $EndComp
 $Comp
-L 3V3 #PWR057
+L 3V3 #PWR064
 U 1 1 522056F5
 P 5950 6600
-F 0 "#PWR057" H 5950 6700 40  0001 C CNN
+F 0 "#PWR064" H 5950 6700 40  0001 C CNN
 F 1 "3V3" H 5950 6725 40  0000 C CNN
 F 2 "" H 5950 6600 60  0001 C CNN
@@
 32MHZ-OSC_EN
 $Comp
-L GNDPWR #PWR058
+L GNDPWR #PWR065
 U 1 1 52DFFE37
 P 10900 2500
-F 0 "#PWR058" H 10900 2550 40  0001 C CNN
+F 0 "#PWR065" H 10900 2550 40  0001 C CNN
 F 1 "GNDPWR" H 10900 2420 40  0000 C CNN
 F 2 "" H 10900 2500 60  0001 C CNN
@@
 $EndComp
 $Comp
-L CSMALL C39
-U 1 1 52FD2767
-P 1500 1250
-F 0 "C39" H 1525 1300 30  0000 L CNN
-F 1 "1n" H 1525 1200 30  0000 L CNN
-F 2 "" H 1500 1250 60  0000 C CNN
-F 3 "" H 1500 1250 60  0000 C CNN
-	1    1500 1250
-	1    0    0    -1
-$EndComp
-$Comp
 L CSMALL C38
 U 1 1 52FD276D
@@
 $EndComp
 $Comp
-L GNDPWR #PWR059
+L GNDPWR #PWR066
 U 1 1 52FD2A0A
 P 1050 1450
-F 0 "#PWR059" H 1050 1500 40  0001 C CNN
+F 0 "#PWR066" H 1050 1500 40  0001 C CNN
 F 1 "GNDPWR" H 1050 1370 40  0000 C CNN
 F 2 "" H 1050 1450 60  0001 C CNN
@@
 F 3 "" H 1200 800 60  0000 C CNN
 	1    1200 800
-	1    0    0    -1
+	-1   0    0    1
 $EndComp
 Text GLabel 1450 1700 0    60   Input ~ 0
@@
 I2C_SDA
 $Comp
-L 3V3 #PWR060
+L 3V3 #PWR067
 U 1 1 52FDE4F8
 P 10400 6000
-F 0 "#PWR060" H 10400 6100 40  0001 C CNN
+F 0 "#PWR067" H 10400 6100 40  0001 C CNN
 F 1 "3V3" H 10400 6125 40  0000 C CNN
 F 2 "" H 10400 6000 60  0001 C CNN
@@
 $EndComp
 $Comp
-L GNDPWR #PWR061
+L GNDPWR #PWR068
 U 1 1 52FDE4FE
 P 10400 6400
-F 0 "#PWR061" H 10400 6450 40  0001 C CNN
+F 0 "#PWR068" H 10400 6450 40  0001 C CNN
 F 1 "GNDPWR" H 10400 6320 40  0000 C CNN
 F 2 "" H 10400 6400 60  0001 C CNN
@@
 $EndComp
 $Comp
-L 3V3 #PWR062
+L 3V3 #PWR069
 U 1 1 52FDE731
 P 10400 5200
-F 0 "#PWR062" H 10400 5300 40  0001 C CNN
+F 0 "#PWR069" H 10400 5300 40  0001 C CNN
 F 1 "3V3" H 10400 5325 40  0000 C CNN
 F 2 "" H 10400 5200 60  0001 C CNN
@@
 $EndComp
 $Comp
-L GNDPWR #PWR063
+L GNDPWR #PWR070
 U 1 1 52FDE737
 P 10400 5600
-F 0 "#PWR063" H 10400 5650 40  0001 C CNN
+F 0 "#PWR070" H 10400 5650 40  0001 C CNN
 F 1 "GNDPWR" H 10400 5520 40  0000 C CNN
 F 2 "" H 10400 5600 60  0001 C CNN
@@
 Connection ~ 850  4900
 Wire Wire Line
-	1500 5050 1500 5100
+	1550 5100 1550 5150
 Wire Wire Line
 	1650 3900 1900 3900
@@
 	1050 1350 1050 1450
 Wire Wire Line
-	1050 1400 1500 1400
-Wire Wire Line
 	1300 1400 1300 1350
 Connection ~ 1050 1400
 Wire Wire Line
-	1500 1400 1500 1350
-Connection ~ 1300 1400
-Wire Wire Line
 	1300 1050 1300 1150
-Wire Wire Line
-	1500 1050 1500 1150
-Connection ~ 1500 1050
 Wire Wire Line
 	1700 800  1550 800
@@
 	5200 6050 5150 6050
 $Comp
-L 3V3 #PWR064
+L 3V3 #PWR071
 U 1 1 52FDEED0
 P 10400 3900
-F 0 "#PWR064" H 10400 4000 40  0001 C CNN
+F 0 "#PWR071" H 10400 4000 40  0001 C CNN
 F 1 "3V3" H 10400 4025 40  0000 C CNN
 F 2 "" H 10400 3900 60  0001 C CNN
@@
 $EndComp
 $Comp
-L GNDPWR #PWR065
+L GNDPWR #PWR072
 U 1 1 52FDEED6
 P 10400 4800
-F 0 "#PWR065" H 10400 4850 40  0001 C CNN
+F 0 "#PWR072" H 10400 4850 40  0001 C CNN
 F 1 "GNDPWR" H 10400 4720 40  0000 C CNN
 F 2 "" H 10400 4800 60  0001 C CNN
@@
 	10350 4050 10500 4050
 $Comp
-L 3V3 #PWR066
+L 3V3 #PWR073
 U 1 1 52FDF3BC
 P 10350 3000
-F 0 "#PWR066" H 10350 3100 40  0001 C CNN
+F 0 "#PWR073" H 10350 3100 40  0001 C CNN
 F 1 "3V3" H 10350 3125 40  0000 C CNN
 F 2 "" H 10350 3000 60  0001 C CNN
@@
 $EndComp
 $Comp
-L GNDPWR #PWR067
+L GNDPWR #PWR074
 U 1 1 52FDF3C2
 P 10350 3500
-F 0 "#PWR067" H 10350 3550 40  0001 C CNN
+F 0 "#PWR074" H 10350 3550 40  0001 C CNN
 F 1 "GNDPWR" H 10350 3420 40  0000 C CNN
 F 2 "" H 10350 3500 60  0001 C CNN
@@
 	900  6550 1000 6550
 $Comp
-L 3V3 #PWR068
+L 3V3 #PWR075
 U 1 1 52FE19DB
 P 600 6100
-F 0 "#PWR068" H 600 6200 40  0001 C CNN
+F 0 "#PWR075" H 600 6200 40  0001 C CNN
 F 1 "3V3" H 600 6225 40  0000 C CNN
 F 2 "" H 600 6100 60  0001 C CNN
@@
 DSP_WAKEUP
 Wire Wire Line
-	1500 4850 1500 4800
-Wire Wire Line
-	1500 4800 1750 4800
-Wire Wire Line
 	1750 5200 1900 5200
 Wire Wire Line
@@
 L RSML R48
 U 1 1 530C94CF
-P 1750 5000
-F 0 "R48" V 1830 5000 40  0000 C CNN
-F 1 "0" V 1752 5000 40  0000 C CNN
-F 2 "" V 1680 5000 30  0000 C CNN
-F 3 "" H 1750 5000 30  0000 C CNN
-	1    1750 5000
-	1    0    0    -1
-$EndComp
-Wire Wire Line
-	1750 5200 1750 5150
-Wire Wire Line
-	1750 4800 1750 4850
+P 1500 4750
+F 0 "R48" V 1580 4750 40  0000 C CNN
+F 1 "0" V 1502 4750 40  0000 C CNN
+F 2 "" V 1430 4750 30  0000 C CNN
+F 3 "" H 1500 4750 30  0000 C CNN
+	1    1500 4750
+	0    -1   -1   0
+$EndComp
+Wire Wire Line
+	1750 4750 1750 5200
 Wire Wire Line
 	5250 6650 5250 6400
@@
 Wire Wire Line
 	1200 3700 1900 3700
+Wire Wire Line
+	1300 4700 1300 4750
+Wire Wire Line
+	1300 4750 1350 4750
+Wire Wire Line
+	1650 4750 1750 4750
+Wire Wire Line
+	1550 4900 1550 4850
+Wire Wire Line
+	1550 4850 1750 4850
+Connection ~ 1750 4850
+Wire Wire Line
+	1050 1400 1300 1400
+$Comp
+L SI7020 U3
+U 1 1 53160704
+P 7300 1600
+F 0 "U3" H 7300 1700 60  0000 C CNN
+F 1 "SI7020" H 7300 1500 60  0000 C CNN
+F 2 "" H 7300 1600 60  0000 C CNN
+F 3 "" H 7300 1600 60  0000 C CNN
+	1    7300 1600
+	1    0    0    -1
+$EndComp
+Text GLabel 7800 1350 1    60   Input ~ 0
+I2C_SCL
+Text GLabel 6800 1350 1    60   Input ~ 0
+I2C_SDA
+$Comp
+L 3V3 #PWR076
+U 1 1 53160713
+P 8050 1200
+F 0 "#PWR076" H 8050 1300 40  0001 C CNN
+F 1 "3V3" H 8050 1325 40  0000 C CNN
+F 2 "" H 8050 1200 60  0001 C CNN
+F 3 "" H 8050 1200 60  0001 C CNN
+	1    8050 1200
+	1    0    0    -1
+$EndComp
+$Comp
+L GNDPWR #PWR077
+U 1 1 53160719
+P 6600 1700
+F 0 "#PWR077" H 6600 1750 40  0001 C CNN
+F 1 "GNDPWR" H 6600 1620 40  0000 C CNN
+F 2 "" H 6600 1700 60  0001 C CNN
+F 3 "" H 6600 1700 60  0001 C CNN
+	1    6600 1700
+	1    0    0    -1
+$EndComp
+NoConn ~ 6800 1750
+NoConn ~ 7800 1750
+Wire Wire Line
+	7800 1350 7800 1450
+Wire Wire Line
+	6800 1350 6800 1450
+Wire Wire Line
+	6600 1700 6600 1600
+Wire Wire Line
+	6600 1600 6800 1600
+$Comp
+L RSML R54
+U 1 1 53160985
+P 8050 1400
+F 0 "R54" V 8130 1400 40  0000 C CNN
+F 1 "0" V 8052 1400 40  0000 C CNN
+F 2 "" V 7980 1400 30  0000 C CNN
+F 3 "" H 8050 1400 30  0000 C CNN
+	1    8050 1400
+	1    0    0    -1
+$EndComp
+$Comp
+L CSMALL C29
+U 1 1 5316099F
+P 8050 1750
+F 0 "C29" H 8075 1800 30  0000 L CNN
+F 1 "100n" H 8075 1700 30  0000 L CNN
+F 2 "" H 8050 1750 60  0000 C CNN
+F 3 "" H 8050 1750 60  0000 C CNN
+	1    8050 1750
+	1    0    0    -1
+$EndComp
+$Comp
+L GNDPWR #PWR078
+U 1 1 531609CD
+P 8050 1900
+F 0 "#PWR078" H 8050 1950 40  0001 C CNN
+F 1 "GNDPWR" H 8050 1820 40  0000 C CNN
+F 2 "" H 8050 1900 60  0001 C CNN
+F 3 "" H 8050 1900 60  0001 C CNN
+	1    8050 1900
+	1    0    0    -1
+$EndComp
+Wire Wire Line
+	7800 1600 8050 1600
+Wire Wire Line
+	8050 1550 8050 1650
+Connection ~ 8050 1600
+Wire Wire Line
+	8050 1850 8050 1900
+Wire Wire Line
+	8050 1200 8050 1250
 $EndSCHEMATC

Commit message: Schematic and board complete (add tps60125 charge-pump, tps77533 LDO regolator, oled).
Parts:
- removed C25: 1u, symbol CSMALL
- removed C30: 10u, symbol CP1SMALL
- removed D2, D3, D4: LED, symbol LED
- removed JP2: LED-DEBUG, symbol JUMPER
- removed P15: GPIOS, symbol CONN_5
- removed P16: SPI, symbol CONN_9
- removed R16: NO, symbol RSML
- removed R28, R32: 220, symbol RSML
- added BTB1: BH411-1P, symbol BH2466
- added BTB2: 1V3, symbol BATTERY
- added C25: 1u, symbol CBIG
- added C30: 10u, symbol CBIG
- added C65, C66: 100n, symbol CSMALL
- added C67: 1u, symbol CSMALL
- added C68: 1u, symbol CP1SMALL
- added P10: DSP-SDA, symbol CONN_1
- added P15: CONN_6, symbol CONN_6
- added P16: SPI, symbol CONN_8
- added PB1: PROG, symbol PUSH-BT_4
- added PB3: WAKEUP, symbol PUSH-BT_4
- added R1, R15, R58: 0, symbol RSML
- added R55, R57: 10K, symbol RSML
- added R56: 220, symbol RSML
- added SW2: JS202011SCQN, symbol JS202011SCQN
- added U10: SST25PF080B, symbol SST25PF080B
- added U13: MCCOG21605B6W, symbol MCCOG21605B6W
- D0: value NO -> LED
- R49: value 220 -> NO
- renumbered PBT2 to PB2
Connections:
- net labels added: 3V3_STEPUP, GPIO3, LED0, SD1_EN, SD2_EN, SPI_CS-FLASH, STEPUP_EN
- net labels removed: GPIO0, LED2, LED3, LED4, SPI_CS0
- wire segments 167 -> 225
Other:
- note added: "BIOS BATTERY(RTC)"
- moved on the sheet: D1, P17, P18, PB2, R27, R54, U3

Commit message: gerber and schematic modified, sendt to MCE
Parts:
- removed P10: DSP-SDA, symbol CONN_1
- P15: value CONN_6 -> GPIOS
- P21: value DSP-SDA -> DSP-CLKOUT
Changed lines of the file:
@@
 NoConn ~ 1900 1900
 $Comp
-L GNDPWR #PWR047
+L GNDPWR #PWR048
 U 1 1 521E22FA
 P 1400 2150
-F 0 "#PWR047" H 1400 2200 40  0001 C CNN
+F 0 "#PWR048" H 1400 2200 40  0001 C CNN
 F 1 "GNDPWR" H 1400 2070 40  0000 C CNN
 F 2 "" H 1400 2150 60  0001 C CNN
@@
 $EndComp
 $Comp
-L 3V3 #PWR048
+L 3V3 #PWR049
 U 1 1 521E2923
 P 850 5750
-F 0 "#PWR048" H 850 5850 40  0001 C CNN
+F 0 "#PWR049" H 850 5850 40  0001 C CNN
 F 1 "3V3" H 850 5875 40  0000 C CNN
 F 2 "" H 850 5750 60  0001 C CNN
@@
 $EndComp
 $Comp
-L GNDPWR #PWR049
+L GNDPWR #PWR050
 U 1 1 521E2CF9
 P 1850 5950
-F 0 "#PWR049" H 1850 6000 40  0001 C CNN
+F 0 "#PWR050" H 1850 6000 40  0001 C CNN
 F 1 "GNDPWR" H 1850 5870 40  0000 C CNN
 F 2 "" H 1850 5950 60  0001 C CNN
@@
 $EndComp
 $Comp
-L GNDPWR #PWR050
+L GNDPWR #PWR051
 U 1 1 521E2F5E
 P 1100 5300
-F 0 "#PWR050" H 1100 5350 40  0001 C CNN
+F 0 "#PWR051" H 1100 5350 40  0001 C CNN
 F 1 "GNDPWR" H 1100 5220 40  0000 C CNN
 F 2 "" H 1100 5300 60  0001 C CNN
@@
 $EndComp
 $Comp
-L 3V3 #PWR051
+L 3V3 #PWR052
 U 1 1 521E31D9
 P 1300 4700
-F 0 "#PWR051" H 1300 4800 40  0001 C CNN
+F 0 "#PWR052" H 1300 4800 40  0001 C CNN
 F 1 "3V3" H 1300 4825 40  0000 C CNN
 F 2 "" H 1300 4700 60  0001 C CNN
@@
 $EndComp
 $Comp
-L GNDPWR #PWR052
+L GNDPWR #PWR053
 U 1 1 521E31DF
 P 1550 5150
-F 0 "#PWR052" H 1550 5200 40  0001 C CNN
+F 0 "#PWR053" H 1550 5200 40  0001 C CNN
 F 1 "GNDPWR" H 1550 5070 40  0000 C CNN
 F 2 "" H 1550 5150 60  0001 C CNN
@@
 NoConn ~ 1900 4900
 $Comp
-L GNDPWR #PWR053
+L GNDPWR #PWR054
 U 1 1 521E336E
 P 1400 4350
-F 0 "#PWR053" H 1400 4400 40  0001 C CNN
+F 0 "#PWR054" H 1400 4400 40  0001 C CNN
 F 1 "GNDPWR" H 1400 4270 40  0000 C CNN
 F 2 "" H 1400 4350 60  0001 C CNN
@@
 $EndComp
 $Comp
-L 3V3 #PWR054
+L 3V3 #PWR055
 U 1 1 522056F5
 P 5950 6600
-F 0 "#PWR054" H 5950 6700 40  0001 C CNN
+F 0 "#PWR055" H 5950 6700 40  0001 C CNN
 F 1 "3V3" H 5950 6725 40  0000 C CNN
 F 2 "" H 5950 6600 60  0001 C CNN
@@
 32MHZ-OSC_EN
 $Comp
-L GNDPWR #PWR055
+L GNDPWR #PWR056
 U 1 1 52DFFE37
 P 9850 1600
-F 0 "#PWR055" H 9850 1650 40  0001 C CNN
+F 0 "#PWR056" H 9850 1650 40  0001 C CNN
 F 1 "GNDPWR" H 9850 1520 40  0000 C CNN
 F 2 "" H 9850 1600 60  0001 C CNN
@@
 $EndComp
 $Comp
-L GNDPWR #PWR056
+L GNDPWR #PWR057
 U 1 1 52FD2A0A
 P 1050 1450
-F 0 "#PWR056" H 1050 1500 40  0001 C CNN
+F 0 "#PWR057" H 1050 1500 40  0001 C CNN
 F 1 "GNDPWR" H 1050 1370 40  0000 C CNN
 F 2 "" H 1050 1450 60  0001 C CNN
@@
 I2C_SDA
 $Comp
-L 3V3 #PWR057
+L 3V3 #PWR058
 U 1 1 52FDE4F8
 P 10400 6300
-F 0 "#PWR057" H 10400 6400 40  0001 C CNN
+F 0 "#PWR058" H 10400 6400 40  0001 C CNN
 F 1 "3V3" H 10400 6425 40  0000 C CNN
 F 2 "" H 10400 6300 60  0001 C CNN
@@
 $EndComp
 $Comp
-L GNDPWR #PWR058
+L GNDPWR #PWR059
 U 1 1 52FDE4FE
 P 10400 6700
-F 0 "#PWR058" H 10400 6750 40  0001 C CNN
+F 0 "#PWR059" H 10400 6750 40  0001 C CNN
 F 1 "GNDPWR" H 10400 6620 40  0000 C CNN
 F 2 "" H 10400 6700 60  0001 C CNN
@@
 $EndComp
 $Comp
-L 3V3 #PWR059
+L 3V3 #PWR060
 U 1 1 52FDE731
 P 10400 5500
-F 0 "#PWR059" H 10400 5600 40  0001 C CNN
+F 0 "#PWR060" H 10400 5600 40  0001 C CNN
 F 1 "3V3" H 10400 5625 40  0000 C CNN
 F 2 "" H 10400 5500 60  0001 C CNN
@@
 $EndComp
 $Comp
-L GNDPWR #PWR060
+L GNDPWR #PWR061
 U 1 1 52FDE737
 P 10400 5900
-F 0 "#PWR060" H 10400 5950 40  0001 C CNN
+F 0 "#PWR061" H 10400 5950 40  0001 C CNN
 F 1 "GNDPWR" H 10400 5820 40  0000 C CNN
 F 2 "" H 10400 5900 60  0001 C CNN
@@
 $EndComp
 $Comp
-L 3V3 #PWR061
+L 3V3 #PWR062
 U 1 1 52FDEED0
 P 10400 4200
-F 0 "#PWR061" H 10400 4300 40  0001 C CNN
+F 0 "#PWR062" H 10400 4300 40  0001 C CNN
 F 1 "3V3" H 10400 4325 40  0000 C CNN
 F 2 "" H 10400 4200 60  0001 C CNN
@@
 $EndComp
 $Comp
-L GNDPWR #PWR062
+L GNDPWR #PWR063
 U 1 1 52FDEED6
 P 10400 5000
-F 0 "#PWR062" H 10400 5050 40  0001 C CNN
+F 0 "#PWR063" H 10400 5050 40  0001 C CNN
 F 1 "GNDPWR" H 10400 4920 40  0000 C CNN
 F 2 "" H 10400 5000 60  0001 C CNN
@@
 SPI_CS2
 $Comp
-L 3V3 #PWR063
+L 3V3 #PWR064
 U 1 1 52FDF3BC
 P 10400 3300
-F 0 "#PWR063" H 10400 3400 40  0001 C CNN
+F 0 "#PWR064" H 10400 3400 40  0001 C CNN
 F 1 "3V3" H 10400 3425 40  0000 C CNN
 F 2 "" H 10400 3300 60  0001 C CNN
@@
 $EndComp
 $Comp
-L GNDPWR #PWR064
+L GNDPWR #PWR065
 U 1 1 52FDF3C2
 P 10400 3900
-F 0 "#PWR064" H 10400 3950 40  0001 C CNN
+F 0 "#PWR065" H 10400 3950 40  0001 C CNN
 F 1 "GNDPWR" H 10400 3820 40  0000 C CNN
 F 2 "" H 10400 3900 60  0001 C CNN
@@
 LED1
 $Comp
-L 3V3 #PWR065
+L 3V3 #PWR066
 U 1 1 52FE19DB
 P 600 6100
-F 0 "#PWR065" H 600 6200 40  0001 C CNN
+F 0 "#PWR066" H 600 6200 40  0001 C CNN
 F 1 "3V3" H 600 6225 40  0000 C CNN
 F 2 "" H 600 6100 60  0001 C CNN
@@
 P 1050 3700
 F 0 "P21" H 1130 3700 40  0000 L CNN
-F 1 "DSP-SDA" H 1050 3755 30  0001 C CNN
+F 1 "DSP-CLKOUT" H 1050 3755 30  0001 C CNN
 F 2 "" H 1050 3700 60  0000 C CNN
 F 3 "" H 1050 3700 60  0000 C CNN
@@
 I2C_SDA
 $Comp
-L 3V3 #PWR066
+L 3V3 #PWR067
 U 1 1 53160713
 P 10850 2150
-F 0 "#PWR066" H 10850 2250 40  0001 C CNN
+F 0 "#PWR067" H 10850 2250 40  0001 C CNN
 F 1 "3V3" H 10850 2275 40  0000 C CNN
 F 2 "" H 10850 2150 60  0001 C CNN
@@
 $EndComp
 $Comp
-L GNDPWR #PWR067
+L GNDPWR #PWR068
 U 1 1 53160719
 P 9400 2650
-F 0 "#PWR067" H 9400 2700 40  0001 C CNN
+F 0 "#PWR068" H 9400 2700 40  0001 C CNN
 F 1 "GNDPWR" H 9400 2570 40  0000 C CNN
 F 2 "" H 9400 2650 60  0001 C CNN
@@
 $EndComp
 $Comp
-L GNDPWR #PWR068
+L GNDPWR #PWR069
 U 1 1 531609CD
 P 10850 2850
-F 0 "#PWR068" H 10850 2900 40  0001 C CNN
+F 0 "#PWR069" H 10850 2900 40  0001 C CNN
 F 1 "GNDPWR" H 10850 2770 40  0000 C CNN
 F 2 "" H 10850 2850 60  0001 C CNN
@@
 $EndComp
 $Comp
-L GNDPWR #PWR069
+L GNDPWR #PWR070
 U 1 1 535E1D3B
 P 4850 7550
-F 0 "#PWR069" H 4850 7600 40  0001 C CNN
+F 0 "#PWR070" H 4850 7600 40  0001 C CNN
 F 1 "GNDPWR" H 4850 7470 40  0000 C CNN
 F 2 "" H 4850 7550 60  0001 C CNN
@@
 Text Notes 3550 6850 0    60   ~ 0
 BIOS BATTERY(RTC)
-$Comp
-L CONN_1 P10
-U 1 1 535E1D43
-P 2950 7500
-F 0 "P10" H 3030 7500 40  0000 L CNN
-F 1 "DSP-SDA" H 2950 7555 30  0001 C CNN
-F 2 "" H 2950 7500 60  0000 C CNN
-F 3 "" H 2950 7500 60  0000 C CNN
-	1    2950 7500
-	-1   0    0    1
-$EndComp
 $Comp
 L BH2466 BTB1
@@
 $EndComp
 $Comp
-L GNDPWR #PWR070
+L GNDPWR #PWR071
 U 1 1 5368FA66
 P 6950 4150
-F 0 "#PWR070" H 6950 4200 40  0001 C CNN
+F 0 "#PWR071" H 6950 4200 40  0001 C CNN
 F 1 "GNDPWR" H 6950 4070 40  0000 C CNN
 F 2 "" H 6950 4150 60  0001 C CNN
@@
 $EndComp
 $Comp
-L 3V3 #PWR071
+L 3V3 #PWR072
 U 1 1 5368FB37
 P 9100 2850
-F 0 "#PWR071" H 9100 2950 40  0001 C CNN
+F 0 "#PWR072" H 9100 2950 40  0001 C CNN
 F 1 "3V3" H 9100 2975 40  0000 C CNN
 F 2 "" H 9100 2850 60  0001 C CNN
@@
 $EndComp
 $Comp
-L GNDPWR #PWR072
+L GNDPWR #PWR073
 U 1 1 5368FB49
 P 8850 3500
-F 0 "#PWR072" H 8850 3550 40  0001 C CNN
+F 0 "#PWR073" H 8850 3550 40  0001 C CNN
 F 1 "GNDPWR" H 8850 3420 40  0000 C CNN
 F 2 "" H 8850 3500 60  0001 C CNN
@@
 $EndComp
 $Comp
-L GNDPWR #PWR073
+L GNDPWR #PWR074
 U 1 1 5369021A
 P 9600 3850
-F 0 "#PWR073" H 9600 3900 40  0001 C CNN
+F 0 "#PWR074" H 9600 3900 40  0001 C CNN
 F 1 "GNDPWR" H 9600 3770 40  0000 C CNN
 F 2 "" H 9600 3850 60  0001 C CNN
@@
 Text GLabel 7000 850  0    60   Input ~ 0
 LED0
-$Comp
-L GNDPWR #PWR074
-U 1 1 536A34AD
-P 2450 7300
-F 0 "#PWR074" H 2450 7350 40  0001 C CNN
-F 1 "GNDPWR" H 2450 7220 40  0000 C CNN
-F 2 "" H 2450 7300 60  0001 C CNN
-F 3 "" H 2450 7300 60  0001 C CNN
-	1    2450 7300
-	1    0    0    -1
-$EndComp
 Text GLabel 1500 7200 0    60   Input ~ 0
 DSP_WAKEUP
@@
 	3250 7050 3100 7050
 Wire Wire Line
-	3100 7500 3700 7500
-Wire Wire Line
 	3250 7050 3250 7500
-Connection ~ 3250 7500
 Wire Wire Line
 	4300 7500 4850 7500
@@
 Wire Wire Line
 	2250 7200 2450 7200
-Wire Wire Line
-	2450 7200 2450 7300
 Wire Wire Line
 	1500 7200 1650 7200
@@
 P 10850 3600
 F 0 "P15" V 10800 3600 60  0000 C CNN
-F 1 "CONN_6" V 10900 3600 60  0000 C CNN
+F 1 "GPIOS" V 10900 3600 60  0000 C CNN
 F 2 "" H 10850 3600 60  0000 C CNN
 F 3 "" H 10850 3600 60  0000 C CNN
@@
 Wire Wire Line
 	9100 1300 9200 1300
+Wire Wire Line
+	3250 7500 3700 7500
+$Comp
+L 3V3 #PWR077
+U 1 1 5385A7D7
+P 2450 7150
+F 0 "#PWR077" H 2450 7250 40  0001 C CNN
+F 1 "3V3" H 2450 7275 40  0000 C CNN
+F 2 "" H 2450 7150 60  0001 C CNN
+F 3 "" H 2450 7150 60  0001 C CNN
+	1    2450 7150
+	1    0    0    -1
+$EndComp
+Wire Wire Line
+	2450 7200 2450 7150
 $EndSCHEMATC
