File: AudioDSP/VirtualSense_ADSP_3.sch (KiCad schematic (older format))
At the start: 21 parts, among them U5 C5535

Commit message: create schematics, components footprints, board layout.
Parts:
- removed SD2: MICRO_SD, symbol MICRO_SD
- added C40, C42: 1u, symbol CP1SMALL
- added C41, C43, C52, C53, C54, C58: 10u, symbol CP1SMALL
- added C44, C45, C46, C47, C55, C56, C57, C60: 100n, symbol CSMALL
- added C48, C49, C51: 1n, symbol CSMALL
- added C50: 10n, symbol CSMALL
- added L5, L6, L7, L8: BLM18AG601SN1D, symbol FILTER
- added P19: DSP-SDA, symbol CONN_1
- added R36, R38, R42, R44, R46: 10K, symbol RSML
- added R40: NO, symbol RSML
- added R50, R51, R52, R53: 0, symbol RSML
- added SD1: SD, symbol MICRO_SD
- added uSD1, uSD2: uSD, symbol CONN_8
- SD2: renamed from SD1; value MICRO_SD -> SD
- gave numbers to parts that had none: 8
Connections:
- net labels added: 3V3_USB, SD1_CLK, SD1_CMD, SD1_DATA0, SD1_DATA1, SD1_DATA2, SD1_DATA3, SD2_CLK, SD2_CMD, SD2_DATA0, SD2_DATA1, SD2_DATA2, SD2_DATA3, USB_LDO_OUT
- net labels removed: SD_CLK, SD_CMD, SD_DATA0, SD_DATA1, SD_DATA2, SD_DATA3, V3.3A
- wire segments 131 -> 235
- no-connect marks 1 -> 0
Other:
- moved on the sheet: C59, R29, R30, R31, R37, R39, R41, R43, R45, R47, SD2, U5B

Commit message: add too many libraries on schematics, board disposal almolst complete, hope that will be routed
Parts:
- removed C48, C49, C51: 1n, symbol CSMALL
- removed C50: 10n, symbol CSMALL
- added uSD1-1: uSD1-1, symbol CONN_8
Connections:
- wire segments 235 -> 236
Other:
- note added: "micro SD package portatile"

Commit message: Schematic and board complete (add tps60125 charge-pump, tps77533 LDO regolator, oled).
Parts:
- removed C40, C42: 1u, symbol CP1SMALL
- removed C41, C43, C52, C53, C54, C58, C59: 10u, symbol CP1SMALL
- removed C57: 100n, symbol CSMALL
- removed R52, R53: 0, symbol RSML
- removed uSD1, uSD2: uSD, symbol CONN_8
- removed uSD1-1: uSD1-1, symbol CONN_8
- added C13, C39, C48, C70, C8: 100n, symbol CSMALL
- added C40, C42: 1u, symbol CBIG
- added C41, C43, C52, C53, C58, C59: 10u, symbol CBIG
- added C49, C50: 100u, symbol CP1
- added C51, C64: 22u, symbol C
- added C62, C63: 2u2, symbol C
- added L10, L11, L12, L9: BLM21BB221SN1D, symbol FILTER
- added R2: 10K, symbol RSML
- added U8: TPS2080D, symbol TPS2080D
- added U9: TPS60125, symbol TPS60125
Connections:
- net labels added: 3V3_STEPUP, SD1_EN, SD1_VCC, SD2_EN, SD2_VCC, STEPUP_EN
- wire segments 236 -> 272
- no-connect marks 0 -> 2
Other:
- note removed: "micro SD package portatile"
- moved on the sheet: R36, R37, R38, R39, R40, R41, R42, R43, R44, R45, R46, R47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

Commit message: gerber and schematic modified, sendt to MCE
Parts:
- P19: value DSP-SDA -> DSP-LDOO
Changed lines of the file:
@@
 $EndComp
 $Comp
-L GNDPWR #PWR026
+L GNDPWR #PWR027
 U 1 1 521E3C9E
 P 6150 6250
-AR Path="/521CC8CD/521E3C9E" Ref="#PWR026"  Part="1"
+AR Path="/521CC8CD/521E3C9E" Ref="#PWR027"  Part="1"
 AR Path="/530DD493/521E3C9E" Ref="#PWR049"  Part="1"
-F 0 "#PWR026" H 6150 6300 40  0001 C CNN
+F 0 "#PWR027" H 6150 6300 40  0001 C CNN
 F 1 "GNDPWR" H 6150 6170 40  0000 C CNN
 F 2 "" H 6150 6250 60  0001 C CNN
@@
 $EndComp
 $Comp
-L GNDPWR #PWR027
+L GNDPWR #PWR028
 U 1 1 521E4612
 P 2000 5400
-AR Path="/521CC8CD/521E4612" Ref="#PWR027"  Part="1"
+AR Path="/521CC8CD/521E4612" Ref="#PWR028"  Part="1"
 AR Path="/530DD493/521E4612" Ref="#PWR050"  Part="1"
-F 0 "#PWR027" H 2000 5450 40  0001 C CNN
+F 0 "#PWR028" H 2000 5450 40  0001 C CNN
 F 1 "GNDPWR" H 2000 5320 40  0000 C CNN
 F 2 "" H 2000 5400 60  0001 C CNN
@@
 $EndComp
 $Comp
-L GNDPWR #PWR028
+L GNDPWR #PWR029
 U 1 1 521E4C9D
 P 2700 2850
-AR Path="/521CC8CD/521E4C9D" Ref="#PWR028"  Part="1"
+AR Path="/521CC8CD/521E4C9D" Ref="#PWR029"  Part="1"
 AR Path="/530DD493/521E4C9D" Ref="#PWR051"  Part="1"
-F 0 "#PWR028" H 2700 2900 40  0001 C CNN
+F 0 "#PWR029" H 2700 2900 40  0001 C CNN
 F 1 "GNDPWR" H 2700 2770 40  0000 C CNN
 F 2 "" H 2700 2850 60  0001 C CNN
@@
 DSP_LDOO
 $Comp
-L 3V3 #PWR029
+L 3V3 #PWR030
 U 1 1 521E60B6
 P 6950 3000
-AR Path="/521CC8CD/521E60B6" Ref="#PWR029"  Part="1"
+AR Path="/521CC8CD/521E60B6" Ref="#PWR030"  Part="1"
 AR Path="/530DD493/521E60B6" Ref="#PWR052"  Part="1"
-F 0 "#PWR029" H 6950 3100 40  0001 C CNN
+F 0 "#PWR030" H 6950 3100 40  0001 C CNN
 F 1 "3V3" H 6950 3125 40  0000 C CNN
 F 2 "" H 6950 3000 60  0001 C CNN
@@
 ANA_LDO_OUT
 $Comp
-L GNDPWR #PWR030
+L GNDPWR #PWR031
 U 1 1 52CFCE2F
 P 6900 1500
-AR Path="/521CC8CD/52CFCE2F" Ref="#PWR030"  Part="1"
+AR Path="/521CC8CD/52CFCE2F" Ref="#PWR031"  Part="1"
 AR Path="/530DD493/52CFCE2F" Ref="#PWR053"  Part="1"
-F 0 "#PWR030" H 6900 1550 40  0001 C CNN
+F 0 "#PWR031" H 6900 1550 40  0001 C CNN
 F 1 "GNDPWR" H 6900 1420 40  0000 C CNN
 F 2 "" H 6900 1500 60  0001 C CNN
@@
 $EndComp
 $Comp
-L GNDPWR #PWR031
+L GNDPWR #PWR032
 U 1 1 52FBE78F
 P 10500 5350
-AR Path="/521CC8CD/52FBE78F" Ref="#PWR031"  Part="1"
+AR Path="/521CC8CD/52FBE78F" Ref="#PWR032"  Part="1"
 AR Path="/530DD493/52FBE78F" Ref="#PWR056"  Part="1"
-F 0 "#PWR031" H 10500 5400 40  0001 C CNN
+F 0 "#PWR032" H 10500 5400 40  0001 C CNN
 F 1 "GNDPWR" H 10500 5270 40  0000 C CNN
 F 2 "" H 10500 5350 60  0001 C CNN
@@
 AGND
 $Comp
-L GNDPWR #PWR032
+L GNDPWR #PWR033
 U 1 1 52FE457F
 P 2700 1400
-AR Path="/521CC8CD/52FE457F" Ref="#PWR032"  Part="1"
+AR Path="/521CC8CD/52FE457F" Ref="#PWR033"  Part="1"
 AR Path="/530DD493/52FE457F" Ref="#PWR057"  Part="1"
-F 0 "#PWR032" H 2700 1450 40  0001 C CNN
+F 0 "#PWR033" H 2700 1450 40  0001 C CNN
 F 1 "GNDPWR" H 2700 1320 40  0000 C CNN
 F 2 "" H 2700 1400 60  0001 C CNN
@@
 $EndComp
 $Comp
-L GNDPWR #PWR033
+L GNDPWR #PWR034
 U 1 1 52FE4FB4
 P 1950 1400
-AR Path="/521CC8CD/52FE4FB4" Ref="#PWR033"  Part="1"
+AR Path="/521CC8CD/52FE4FB4" Ref="#PWR034"  Part="1"
 AR Path="/530DD493/52FE4FB4" Ref="#PWR058"  Part="1"
-F 0 "#PWR033" H 1950 1450 40  0001 C CNN
+F 0 "#PWR034" H 1950 1450 40  0001 C CNN
 F 1 "GNDPWR" H 1950 1320 40  0000 C CNN
 F 2 "" H 1950 1400 60  0001 C CNN
@@
 $EndComp
 $Comp
-L GNDPWR #PWR034
+L GNDPWR #PWR035
 U 1 1 52FE71EE
 P 1900 3000
-AR Path="/521CC8CD/52FE71EE" Ref="#PWR034"  Part="1"
+AR Path="/521CC8CD/52FE71EE" Ref="#PWR035"  Part="1"
 AR Path="/530DD493/52FE71EE" Ref="#PWR059"  Part="1"
-F 0 "#PWR034" H 1900 3050 40  0001 C CNN
+F 0 "#PWR035" H 1900 3050 40  0001 C CNN
 F 1 "GNDPWR" H 1900 2920 40  0000 C CNN
 F 2 "" H 1900 3000 60  0001 C CNN
@@
 $EndComp
 $Comp
-L GNDPWR #PWR035
+L GNDPWR #PWR036
 U 1 1 530B3555
 P 6350 3550
-AR Path="/521CC8CD/530B3555" Ref="#PWR035"  Part="1"
+AR Path="/521CC8CD/530B3555" Ref="#PWR036"  Part="1"
 AR Path="/530DD493/530B3555" Ref="#PWR061"  Part="1"
-F 0 "#PWR035" H 6350 3600 40  0001 C CNN
+F 0 "#PWR036" H 6350 3600 40  0001 C CNN
 F 1 "GNDPWR" H 6350 3470 40  0000 C CNN
 F 2 "" H 6350 3550 60  0001 C CNN
@@
 $EndComp
 $Comp
-L GNDPWR #PWR036
+L GNDPWR #PWR037
 U 1 1 530B3F12
 P 6350 2150
-AR Path="/521CC8CD/530B3F12" Ref="#PWR036"  Part="1"
+AR Path="/521CC8CD/530B3F12" Ref="#PWR037"  Part="1"
 AR Path="/530DD493/530B3F12" Ref="#PWR062"  Part="1"
-F 0 "#PWR036" H 6350 2200 40  0001 C CNN
+F 0 "#PWR037" H 6350 2200 40  0001 C CNN
 F 1 "GNDPWR" H 6350 2070 40  0000 C CNN
 F 2 "" H 6350 2150 60  0001 C CNN
@@
 $EndComp
 $Comp
-L GNDPWR #PWR037
+L GNDPWR #PWR038
 U 1 1 530B838A
 P 10500 3100
-AR Path="/521CC8CD/530B838A" Ref="#PWR037"  Part="1"
+AR Path="/521CC8CD/530B838A" Ref="#PWR038"  Part="1"
 AR Path="/530DD493/530B838A" Ref="#PWR064"  Part="1"
-F 0 "#PWR037" H 10500 3150 40  0001 C CNN
+F 0 "#PWR038" H 10500 3150 40  0001 C CNN
 F 1 "GNDPWR" H 10500 3020 40  0000 C CNN
 F 2 "" H 10500 3100 60  0001 C CNN
@@
 SD1_DATA0
 $Comp
-L 3V3 #PWR038
+L 3V3 #PWR039
 U 1 1 530C8AF9
 P 1200 4000
-AR Path="/521CC8CD/530C8AF9" Ref="#PWR038"  Part="1"
+AR Path="/521CC8CD/530C8AF9" Ref="#PWR039"  Part="1"
 AR Path="/530DD493/530C8AF9" Ref="#PWR068"  Part="1"
-F 0 "#PWR038" H 1200 4100 40  0001 C CNN
+F 0 "#PWR039" H 1200 4100 40  0001 C CNN
 F 1 "3V3" H 1200 4125 40  0000 C CNN
 F 2 "" H 1200 4000 60  0001 C CNN
@@
 $EndComp
 $Comp
-L GNDPWR #PWR039
+L GNDPWR #PWR040
 U 1 1 530C8C68
 P 2250 4400
-AR Path="/521CC8CD/530C8C68" Ref="#PWR039"  Part="1"
+AR Path="/521CC8CD/530C8C68" Ref="#PWR040"  Part="1"
 AR Path="/530DD493/530C8C68" Ref="#PWR069"  Part="1"
-F 0 "#PWR039" H 2250 4450 40  0001 C CNN
+F 0 "#PWR040" H 2250 4450 40  0001 C CNN
 F 1 "GNDPWR" H 2250 4320 40  0000 C CNN
 F 2 "" H 2250 4400 60  0001 C CNN
@@
 AR Path="/530DD493/530CAB0D" Ref="P19"  Part="1"
 F 0 "P19" H 6930 1950 40  0000 L CNN
-F 1 "DSP-SDA" H 6850 2005 30  0001 C CNN
+F 1 "DSP-LDOO" H 6850 2005 30  0001 C CNN
 F 2 "" H 6850 1950 60  0000 C CNN
 F 3 "" H 6850 1950 60  0000 C CNN
@@
 $EndComp
 $Comp
-L GNDPWR #PWR040
+L GNDPWR #PWR041
 U 1 1 5369EEB8
 P 3000 7500
-F 0 "#PWR040" H 3000 7550 40  0001 C CNN
+F 0 "#PWR041" H 3000 7550 40  0001 C CNN
 F 1 "GNDPWR" H 3000 7420 40  0000 C CNN
 F 2 "" H 3000 7500 60  0001 C CNN
@@
 $EndComp
 $Comp
-L GNDPWR #PWR041
+L GNDPWR #PWR042
 U 1 1 536A1668
 P 5200 7600
-F 0 "#PWR041" H 5200 7650 40  0001 C CNN
+F 0 "#PWR042" H 5200 7650 40  0001 C CNN
 F 1 "GNDPWR" H 5200 7520 40  0000 C CNN
 F 2 "" H 5200 7600 60  0001 C CNN
@@
 $EndComp
 $Comp
-L GNDPWR #PWR042
+L GNDPWR #PWR043
 U 1 1 536A9A11
 P 10100 2400
-F 0 "#PWR042" H 10100 2450 40  0001 C CNN
+F 0 "#PWR043" H 10100 2450 40  0001 C CNN
 F 1 "GNDPWR" H 10100 2320 40  0000 C CNN
 F 2 "" H 10100 2400 60  0001 C CNN
@@
 3V3_STEPUP
 $Comp
-L 3V3 #PWR043
+L 3V3 #PWR044
 U 1 1 536AC6B3
 P 7950 700
-F 0 "#PWR043" H 7950 800 40  0001 C CNN
+F 0 "#PWR044" H 7950 800 40  0001 C CNN
 F 1 "3V3" H 7950 825 40  0000 C CNN
 F 2 "" H 7950 700 60  0001 C CNN
@@
 NoConn ~ 8900 1050
 $Comp
-L GNDPWR #PWR044
+L GNDPWR #PWR045
 U 1 1 536ACDF9
 P 7950 1300
-F 0 "#PWR044" H 7950 1350 40  0001 C CNN
+F 0 "#PWR045" H 7950 1350 40  0001 C CNN
 F 1 "GNDPWR" H 7950 1220 40  0000 C CNN
 F 2 "" H 7950 1300 60  0001 C CNN
@@
 $EndComp
 $Comp
-L GNDPWR #PWR045
+L GNDPWR #PWR046
 U 1 1 536AD9F7
 P 10550 1250
-F 0 "#PWR045" H 10550 1300 40  0001 C CNN
+F 0 "#PWR046" H 10550 1300 40  0001 C CNN
 F 1 "GNDPWR" H 10550 1170 40  0000 C CNN
 F 2 "" H 10550 1250 60  0001 C CNN
@@
 STEPUP_EN
 $Comp
-L GNDPWR #PWR046
+L GNDPWR #PWR047
 U 1 1 536D0435
 P 3550 6700
-F 0 "#PWR046" H 3550 6750 40  0001 C CNN
+F 0 "#PWR047" H 3550 6750 40  0001 C CNN
 F 1 "GNDPWR" H 3550 6620 40  0000 C CNN
 F 2 "" H 3550 6700 60  0001 C CNN
